Commit message: 修复运控target相关的问题

File: gento_luna_description/xacro/robot.xacro (robot description, xacro)
@@ -1,4 +1,7 @@
 <?xml version="1.0"?>
 <robot name="Gento Luna" xmlns:xacro="http://www.ros.org/wiki/xacro">
+	<!-- topology:=full (default): whole humanoid.
+	     topology:=dual: arms-only tree rooted at arm_base (split_body / demo OCS2 planning). -->
+	<xacro:arg name="topology" default="full"/>
 	<xacro:arg name="collider" default="simple"/>
 	<xacro:arg name="chassis_joints_movable" default="false"/>
@@ -7,10 +10,21 @@
 	<xacro:arg name="right_tcp_offset_xyz" default="0 0 0"/>
 	<xacro:arg name="right_tcp_offset_rpy" default="0 0 0"/>
-	<xacro:include filename="$(find fiveages_w2_common_description)/xacro/components/linkhou_s2_v2.xacro"/>
-	<xacro:linkhou_s2 joints_movable="$(arg chassis_joints_movable)" collider="$(arg collider)"/>
-	<xacro:include filename="$(find gento_luna_description)/xacro/components/torso.xacro"/>
-	<xacro:torso collider="$(arg collider)"/>
-	<xacro:include filename="$(find gento_luna_description)/xacro/components/head.xacro"/>
-	<xacro:head collider="$(arg collider)"/>
+	<xacro:property name="topology_arg" value="$(arg topology)"/>
+	<xacro:unless value="${topology_arg == 'dual'}">
+		<xacro:include filename="$(find fiveages_w2_common_description)/xacro/components/linkhou_s2_v2.xacro"/>
+		<xacro:linkhou_s2 joints_movable="$(arg chassis_joints_movable)" collider="$(arg collider)"/>
+		<xacro:include filename="$(find gento_luna_description)/xacro/components/torso.xacro"/>
+		<xacro:torso collider="$(arg collider)"/>
+		<xacro:include filename="$(find gento_luna_description)/xacro/components/head.xacro"/>
+		<xacro:head collider="$(arg collider)"/>
+	</xacro:unless>
+	<xacro:if value="${topology_arg == 'dual'}">
+		<link name="base_link"/>
+		<link name="arm_base"/>
+		<joint name="arm_base_joint" type="fixed">
+			<parent link="base_link"/>
+			<child link="arm_base"/>
+		</joint>
+	</xacro:if>
 	<!-- CAD J1 at y=±0.2146 z=0.3915 on Leg_J6; M6S Lite joint1 coincides with base_link -->
 	<xacro:include filename="$(find m6_ccs_description)/xacro/arm_mount.xacro"/>

File: gento_skye_description/xacro/robot.xacro (robot description, xacro)
@@ -1,4 +1,7 @@
 <?xml version="1.0"?>
 <robot name="Gento Skye" xmlns:xacro="http://www.ros.org/wiki/xacro">
+	<!-- topology:=full (default): whole humanoid.
+	     topology:=dual: arms-only tree rooted at arm_base (split_body / demo OCS2 planning). -->
+	<xacro:arg name="topology" default="full"/>
 	<xacro:arg name="collider" default="simple"/>
 	<xacro:arg name="chassis_joints_movable" default="false"/>
@@ -11,4 +14,5 @@
 	<xacro:arg name="right_tcp_offset_xyz" default="0 0 0"/>
 	<xacro:arg name="right_tcp_offset_rpy" default="0 0 0"/>
+	<xacro:property name="topology_arg" value="$(arg topology)"/>
 	<xacro:property name="type_arg" value="$(arg type)"/>
 	<xacro:property name="left_type_arg" value="$(arg left_type)"/>
@@ -19,10 +23,20 @@
 	<xacro:set_side_eef_types side="left" type_key="${effective_left_type}"/>
 	<xacro:set_side_eef_types side="right" type_key="${effective_right_type}"/>
-	<xacro:include filename="$(find fiveages_w2_common_description)/xacro/components/linkhou_s2_v2.xacro"/>
-	<xacro:linkhou_s2 joints_movable="$(arg chassis_joints_movable)" collider="$(arg collider)"/>
-	<xacro:include filename="$(find gento_skye_description)/xacro/components/waist.xacro"/>
-	<xacro:waist collider="$(arg collider)"/>
-	<xacro:include filename="$(find gento_skye_description)/xacro/components/head.xacro"/>
-	<xacro:head collider="$(arg collider)"/>
+	<xacro:unless value="${topology_arg == 'dual'}">
+		<xacro:include filename="$(find fiveages_w2_common_description)/xacro/components/linkhou_s2_v2.xacro"/>
+		<xacro:linkhou_s2 joints_movable="$(arg chassis_joints_movable)" collider="$(arg collider)"/>
+		<xacro:include filename="$(find gento_skye_description)/xacro/components/waist.xacro"/>
+		<xacro:waist collider="$(arg collider)"/>
+		<xacro:include filename="$(find gento_skye_description)/xacro/components/head.xacro"/>
+		<xacro:head collider="$(arg collider)"/>
+	</xacro:unless>
+	<xacro:if value="${topology_arg == 'dual'}">
+		<link name="base_link"/>
+		<link name="arm_base"/>
+		<joint name="arm_base_joint" type="fixed">
+			<parent link="base_link"/>
+			<child link="arm_base"/>
+		</joint>
+	</xacro:if>
 	<!-- CAD J1 at y=±0.2305 z=0.4335 on waist_Link_3; M6-CCS joint1 is 0.1745 along base Z
 	     → DualArmMount y = ±(0.2305 - 0.1745) = ±0.056 -->
