Commit message: update xacro

File: gento_luna_description/xacro/component.xacro (robot description, xacro)
@@ -1,15 +1,24 @@
 <?xml version="1.0" ?>
-<robot name="Gento Luna" xmlns:xacro="http://www.ros.org/wiki/xacro">
+<robot name="Luna" xmlns:xacro="http://www.ros.org/wiki/xacro">
+	<!-- Component: head, torso, body (torso + head). isaac:=true hides camera/sensor meshes. -->
 	<xacro:arg name="type" default="head"/>
 	<xacro:arg name="collider" default="simple"/>
+	<xacro:arg name="isaac" default="true"/>
 	<xacro:if value="${'$(arg type)' == 'head'}">
 		<link name="head_mount"/>
 		<xacro:include filename="$(find gento_luna_description)/xacro/components/head.xacro"/>
-		<xacro:head collider="$(arg collider)"/>
+		<xacro:head collider="$(arg collider)" isaac="$(arg isaac)"/>
 	</xacro:if>
 	<xacro:if value="${'$(arg type)' == 'torso'}">
 		<link name="base_link"/>
 		<xacro:include filename="$(find gento_luna_description)/xacro/components/torso.xacro"/>
-		<xacro:torso collider="$(arg collider)"/>
+		<xacro:torso collider="$(arg collider)" isaac="$(arg isaac)"/>
+	</xacro:if>
+	<xacro:if value="${'$(arg type)' == 'body'}">
+		<link name="base_link"/>
+		<xacro:include filename="$(find gento_luna_description)/xacro/components/torso.xacro"/>
+		<xacro:torso collider="$(arg collider)" isaac="$(arg isaac)"/>
+		<xacro:include filename="$(find gento_luna_description)/xacro/components/head.xacro"/>
+		<xacro:head collider="$(arg collider)" isaac="$(arg isaac)"/>
 	</xacro:if>
 </robot>

File: gento_luna_description/xacro/components/head.xacro (robot description, xacro)
@@ -3,5 +3,5 @@
 	<xacro:property name="PI" value="3.1415926535897931"/>
 	<!-- 2-DOF yaw/pitch from Luna CAD. Mount xyz+rpy (incl. +90° about X) is owned by torso. -->
-	<xacro:macro name="head" params="collider:='simple'">
+	<xacro:macro name="head" params="collider:='simple' isaac:=false">
 		<link name="head_link1">
 			<inertial>

File: gento_luna_description/xacro/components/torso.xacro (robot description, xacro)
@@ -4,5 +4,5 @@
 	<!-- 6-DOF torso chain from Gento Luna CAD (Leg_J1–J6).
 	     Creates head_mount (90° pre-rotation absorbed) and arm_base on body_link6. -->
-	<xacro:macro name="torso" params="collider:='simple' parent_link:='base_link' mount_xyz:='0.107 0 0.02'">
+	<xacro:macro name="torso" params="collider:='simple' parent_link:='base_link' mount_xyz:='0.107 0 0.02' isaac:=false">
 		<link name="body_base">
 			<inertial>

File: gento_skye_description/xacro/component.xacro (robot description, xacro)
@@ -1,15 +1,24 @@
 <?xml version="1.0" ?>
-<robot name="Gento Skye" xmlns:xacro="http://www.ros.org/wiki/xacro">
+<robot name="Skye" xmlns:xacro="http://www.ros.org/wiki/xacro">
+	<!-- Component: head, waist, body (waist + head). isaac:=true hides camera/sensor meshes. -->
 	<xacro:arg name="type" default="head"/>
 	<xacro:arg name="collider" default="simple"/>
+	<xacro:arg name="isaac" default="true"/>
 	<xacro:if value="${'$(arg type)' == 'head'}">
 		<link name="head_mount"/>
 		<xacro:include filename="$(find gento_skye_description)/xacro/components/head.xacro"/>
-		<xacro:head collider="$(arg collider)"/>
+		<xacro:head collider="$(arg collider)" isaac="$(arg isaac)"/>
 	</xacro:if>
 	<xacro:if value="${'$(arg type)' == 'waist'}">
 		<link name="base_link"/>
 		<xacro:include filename="$(find gento_skye_description)/xacro/components/waist.xacro"/>
-		<xacro:waist collider="$(arg collider)"/>
+		<xacro:waist collider="$(arg collider)" isaac="$(arg isaac)"/>
+	</xacro:if>
+	<xacro:if value="${'$(arg type)' == 'body'}">
+		<link name="base_link"/>
+		<xacro:include filename="$(find gento_skye_description)/xacro/components/waist.xacro"/>
+		<xacro:waist collider="$(arg collider)" isaac="$(arg isaac)"/>
+		<xacro:include filename="$(find gento_skye_description)/xacro/components/head.xacro"/>
+		<xacro:head collider="$(arg collider)" isaac="$(arg isaac)"/>
 	</xacro:if>
 </robot>

File: gento_skye_description/xacro/components/head.xacro (robot description, xacro)
@@ -3,5 +3,5 @@
 	<xacro:property name="PI" value="3.1415926535897931"/>
 	<!-- 2-DOF yaw/pitch from Skye CAD. Mount xyz (no extra rpy) is owned by waist. -->
-	<xacro:macro name="head" params="collider:='simple'">
+	<xacro:macro name="head" params="collider:='simple' isaac:=false">
 		<link name="head_link1">
 			<inertial>
